File: pcb/rev1/texteditor.kicad_sch (KiCad schematic)
At the start: 17 parts, among them J1 Conn_02x08_Odd_Even, J2 SD_Module, J3 Screw_Terminal_01x02, J4 LED, J5 Conn_01x02, J6 Conn_01x01, J7 Conn_01x03, J8 Conn_01x03, Q1 BC547, SW1 SW_SPDT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

Commit message: rev0.1 -> rev1 pcb
Finalized design since I sent it in for fabrication
Parts:
- J3: value Screw_Terminal_01x02 -> Power In (7v-20v)
- J5: value Conn_01x02 -> Contrast Breakout
- J6: value Conn_01x01 -> LED Potentiometer
Connections:
- net +5V: now also Q1.1 (C)
- net GND: now also J4.2 (Pin_2)
- net CD: now reaches J2.CD (Pin_9)
- net CD: now also U1.15 (GP11)
Other:
- moved on the sheet: J1, J2, J5, J6, Q1, R1
