File: pcb/rev1.1/texteditor.kicad_pcb (KiCad board)
At the start: 2 copper layers, 99.7 x 48.3 mm, 18 parts, among them J1 Conn_02x08_Odd_Even, J2 SD_Module, J3 Power In (7v-20v), J4 LED, J5 Contrast Breakout, J6 LED Potentiometer, J7 Conn_01x03, J8 Conn_01x03, J9 Contrast Potentiometer, Q1 BC547, SW1 SW_SPDT, U2 L7805

Commit message: finish routing, update quote on silkscreen
Routing:
- net +3V3: track 49.5 -> 81.4 mm, vias 2 -> 4
Other:
- board text added: "{dblquote}We don't make mistakes, just happy little accidents.{dblquote} - Bob Ross"
- board text removed: "{dblquote}I can fix a bad page. I can't fix a blank one.{dblquote} - Nora Roberts"
Changed lines of the file:
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@@
 		)
 	)
-	(gr_text "{dblquote}I can fix a bad page.\n I can't fix a blank one.{dblquote}\n	- Nora Roberts"
+	(gr_text "{dblquote}We don't make mistakes,\n just happy little accidents.{dblquote}\n	- Bob Ross"
 		(at 107.95 66.548 0)
 		(layer "F.SilkS")
@@
 	)
 	(segment
+		(start 167.64 61.976)
+		(end 167.64 64.77)
+		(width 0.2)
+		(layer "F.Cu")
+		(net "PWM_BL")
+	)
+	(segment
+		(start 166.116 60.452)
+		(end 167.64 61.976)
+		(width 0.2)
+		(layer "F.Cu")
+		(net "PWM_BL")
+	)
+	(segment
 		(start 187.325 59.375)
 		(end 186.878 58.928)
@@
 		(layer "F.Cu")
 		(net "Net-(Q1-B)")
+	)
+	(segment
+		(start 154.305 92.075)
+		(end 154.305 98.42)
+		(width 0.2)
+		(layer "F.Cu")
+		(net "PWM_CON")
+	)
+	(segment
+		(start 154.305 92.075)
+		(end 155.695 90.685)
+		(width 0.2)
+		(layer "B.Cu")
+		(net "PWM_CON")
+	)
+	(segment
+		(start 158.87 83.026346)
+		(end 158.87 73.54)
+		(width 0.2)
+		(layer "B.Cu")
+		(net "PWM_CON")
+	)
+	(segment
+		(start 155.695 90.685)
+		(end 155.695 86.201346)
+		(width 0.2)
+		(layer "B.Cu")
+		(net "PWM_CON")
+	)
+	(segment
+		(start 158.87 73.54)
+		(end 164.846 67.564)
+		(width 0.2)
+		(layer "B.Cu")
+		(net "PWM_CON")
+	)
+	(segment
+		(start 164.846 67.564)
+		(end 169.926 67.564)
+		(width 0.2)
+		(layer "B.Cu")
+		(net "PWM_CON")
+	)
+	(segment
+		(start 155.695 86.201346)
+		(end 158.87 83.026346)
+		(width 0.2)
+		(layer "B.Cu")
+		(net "PWM_CON")
+	)
+	(segment
+		(start 169.926 67.564)
+		(end 172.72 64.77)
+		(width 0.2)
+		(layer "B.Cu")
+		(net "PWM_CON")
 	)
 	(segment
@@
 	)
 	(segment
+		(start 178.435 84.455)
+		(end 180.34 82.55)
+		(width 0.2)
+		(layer "F.Cu")
+		(net "Net-(J9-Pin_1)")
+	)
+	(segment
+		(start 175.641 84.455)
+		(end 178.435 84.455)
+		(width 0.2)
+		(layer "F.Cu")
+		(net "Net-(J9-Pin_1)")
+	)
+	(segment
+		(start 171.196 88.9)
+		(end 175.641 84.455)
+		(width 0.2)
+		(layer "F.Cu")
+		(net "Net-(J9-Pin_1)")
+	)
+	(segment
+		(start 116.84 64.77)
+		(end 115.316 63.246)
+		(width 0.2)
+		(layer "F.Cu")
+		(net "+3V3")
+	)
+	(segment
+		(start 115.316 63.246)
+		(end 115.316 59.944)
+		(width 0.2)
+		(layer "F.Cu")
+		(net "+3V3")
+	)
+	(segment
 		(start 185.42 82.55)
 		(end 174.625 71.755)
@@
 		(width 0.2)
 		(layer "F.Cu")
+		(net "+3V3")
+	)
+	(segment
+		(start 142.24 67.31)
+		(end 139.7 64.77)
+		(width 0.2)
+		(layer "F.Cu")
+		(net "+3V3")
+	)
+	(segment
+		(start 139.7 64.77)
+		(end 124.46 64.77)
+		(width 0.2)
+		(layer "F.Cu")
+		(net "+3V3")
+	)
+	(via
+		(at 124.46 64.77)
+		(size 0.6)
+		(drill 0.3)
+		(layers "F.Cu" "B.Cu")
 		(net "+3V3")
 	)
@@
 		(net "+3V3")
 	)
+	(via
+		(at 116.84 64.77)
+		(size 0.6)
+		(drill 0.3)
+		(layers "F.Cu" "B.Cu")
+		(net "+3V3")
+	)
 	(segment
 		(start 153.035 71.755)
@@
 	)
 	(segment
+		(start 124.46 64.77)
+		(end 116.84 64.77)
+		(width 0.2)
+		(layer "B.Cu")
+		(net "+3V3")
+	)
+	(segment
+		(start 186.055 60.325)
+		(end 181.229 60.325)
+		(width 0.2)
+		(layer "F.Cu")
+		(net "Net-(J4-Pin_1)")
+	)
+	(segment
+		(start 181.229 60.325)
+		(end 181.102 60.198)
+		(width 0.2)
+		(layer "F.Cu")
+		(net "Net-(J4-Pin_1)")
+	)
+	(segment
 		(start 176.53 101.6)
 		(end 181.61 96.52)
@@
 		(net "Net-(J3-Pin_1)")
 	)
-	(segment
-		(start 167.64 61.976)
-		(end 167.64 64.77)
-		(width 0.2)
-		(layer "F.Cu")
-		(net "PWM_BL")
-	)
-	(segment
-		(start 166.116 60.452)
-		(end 167.64 61.976)
-		(width 0.2)
-		(layer "F.Cu")
-		(net "PWM_BL")
-	)
-	(segment
-		(start 186.055 60.325)
-		(end 181.229 60.325)
-		(width 0.2)
-		(layer "F.Cu")
-		(net "Net-(J4-Pin_1)")
-	)
-	(segment
-		(start 181.229 60.325)
-		(end 181.102 60.198)
-		(width 0.2)
-		(layer "F.Cu")
-		(net "Net-(J4-Pin_1)")
-	)
-	(segment
-		(start 178.435 84.455)
-		(end 180.34 82.55)
-		(width 0.2)
-		(layer "F.Cu")
-		(net "Net-(J9-Pin_1)")
-	)
-	(segment
-		(start 175.641 84.455)
-		(end 178.435 84.455)
-		(width 0.2)
-		(layer "F.Cu")
-		(net "Net-(J9-Pin_1)")
-	)
-	(segment
-		(start 171.196 88.9)
-		(end 175.641 84.455)
-		(width 0.2)
-		(layer "F.Cu")
-		(net "Net-(J9-Pin_1)")
-	)
-	(segment
-		(start 154.305 92.075)
-		(end 154.305 98.42)
-		(width 0.2)
-		(layer "F.Cu")
-		(net "PWM_CON")
-	)
-	(segment
-		(start 154.305 92.075)
-		(end 155.695 90.685)
-		(width 0.2)
-		(layer "B.Cu")
-		(net "PWM_CON")
-	)
-	(segment
-		(start 158.87 83.026346)
-		(end 158.87 73.54)
-		(width 0.2)
-		(layer "B.Cu")
-		(net "PWM_CON")
-	)
-	(segment
-		(start 155.695 90.685)
-		(end 155.695 86.201346)
-		(width 0.2)
-		(layer "B.Cu")
-		(net "PWM_CON")
-	)
-	(segment
-		(start 158.87 73.54)
-		(end 164.846 67.564)
-		(width 0.2)
-		(layer "B.Cu")
-		(net "PWM_CON")
-	)
-	(segment
-		(start 164.846 67.564)
-		(end 169.926 67.564)
-		(width 0.2)
-		(layer "B.Cu")
-		(net "PWM_CON")
-	)
-	(segment
-		(start 155.695 86.201346)
-		(end 158.87 83.026346)
-		(width 0.2)
-		(layer "B.Cu")
-		(net "PWM_CON")
-	)
-	(segment
-		(start 169.926 67.564)
-		(end 172.72 64.77)
-		(width 0.2)
-		(layer "B.Cu")
-		(net "PWM_CON")
-	)
 	(zone

Commit message: Add better headers for potentiometers
Parts:
- removed J6: LED Potentiometer, Connector_PinHeader_2.54mm:PinHeader_1x01_P2.54mm_Vertical
- added J10: Brightness Pot, Connector_PinHeader_2.54mm:PinHeader_1x03_P2.54mm_Vertical, F.Cu at (168.7, 89.5)
- J9: value Contrast Potentiometer -> Contrast Pot; footprint Connector_PinHeader_2.54mm:PinHeader_1x01_P2.54mm_Vertical -> Connector_PinHeader_2.54mm:PinHeader_1x03_P2.54mm_Vertical
- moved J9 6.63 mm to (177.8, 89.5), turned to -90 degrees
- moved J8 5.47 mm to (187.3, 91.3)
- moved J7 5.47 mm to (187.3, 86.6)
Connections:
- J9 pad 1: Net-(J9-Pin_1) -> +3V3
- U1 pad 34: Net-(J9-Pin_1) -> Net-(J9-Pin_2)
Routing:
- net +3V3: track 81.4 -> 102.2 mm
- net Net-(J9-Pin_1): track 11.8 -> 0.00 mm
- net Net-(J9-Pin_2): track 0.00 -> 9.09 mm
- net GND: track 0.00 -> 6.04 mm, vias 0 -> 1
- net Net-(J10-Pin_2): track 12.8 -> 12.0 mm
Other:
- board text added: "Brightness"
- board text removed: "CON pot"
- board text removed: "LED pot"
